File: z80blinken/z80blinken.kicad_sch (KiCad schematic)
At the start: 28 parts, among them J1 RCBus-80, SW1 RESET, SW2 SW_SPST, U1 Z80CPU, U2 4050, U3 4050, U4 MCP100-475D, X1 CXO_DIP8

Commit message: Misc tweaks to boards
Connections:
- no-connect marks 0 -> 38
