File: z80ctrlng/z80ctrlng.kicad_sch (KiCad schematic)
At the start: 33 parts, among them J1 RCBUS, SW1 RESET, SW2 BANK_EN, U1 AS6C4008-55PCN, U2 AVR128DB64x-xPT, U3 74HCT574, U4 74HCT257, U7 AMS1117-3.3

Commit message: Misc tweaks to boards
Changed lines of the file:
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@@
   (bus_alias "BANKBUS" (members "BA[15..18]" "BB[15..18]"))
   (bus_alias "RCBUS" (members "A[0..18]" "A15B" "D[0..15]" "GND" "+5V" "~{M1}" "~{Z80RST}" "Z80CLK" "~{INT}" "~{MREQ}" "~{WR}" "~{RD}" "~{IORQ}" "~{BUSACK}" "~{HALT}" "~{BUSRQ}" "~{WAIT}" "~{NMI}" "TX1B" "RX1B" "TX2B" "RX2B" "BCK"))
+  (junction (at 26.035 168.91) (diameter 0) (color 0 0 0 0)
+  )
   (junction (at 66.675 31.115) (diameter 0) (color 0 0 0 0)
   )
@@
   (junction (at 153.67 19.05) (diameter 0) (color 0 0 0 0)
   )
-  (junction (at 40.64 168.91) (diameter 0) (color 0 0 0 0)
-  )
   (junction (at 238.76 27.94) (diameter 0) (color 0 0 0 0)
   )
@@
     (stroke (width 0) (type default))
   )
-  (wire (pts (xy 45.72 168.91) (xy 40.64 168.91))
-    (stroke (width 0) (type default))
-  )
   (wire (pts (xy 151.13 95.25) (xy 143.51 95.25))
     (stroke (width 0) (type default))
@@
     (stroke (width 0) (type default))
   )
-  (wire (pts (xy 34.925 168.91) (xy 40.64 168.91))
+  (wire (pts (xy 34.925 168.91) (xy 45.72 168.91))
     (stroke (width 0) (type default))
   )
@@
     (stroke (width 0) (type default))
   )
+  (wire (pts (xy 34.925 180.34) (xy 53.34 180.34))
+    (stroke (width 0) (type default))
+  )
   (wire (pts (xy 251.46 74.295) (xy 274.32 74.295))
     (stroke (width 0) (type default))
@@
     (stroke (width 0) (type default))
   )
-  (wire (pts (xy 34.925 180.34) (xy 53.34 180.34))
-    (stroke (width 0) (type default))
-  )
   (bus (pts (xy 120.65 80.01) (xy 120.65 77.47))
     (stroke (width 0) (type default))
@@
     (stroke (width 0) (type default))
   )
+  (text_box "Power Supply"
+    (at 13.335 152.4 0) (size 72.39 36.195)
+    (stroke (width 0) (type dash))
+    (fill (type none))
+    (effects (font (size 1.27 1.27)) (justify left top))
+  )
   (label "A2" (at 274.32 41.275 180) (fields_autoplaced)
     (effects (font (size 1.27 1.27)) (justify right bottom))
@@
     )
   )
-  (symbol (lib_id "power:PWR_FLAG") (at 40.64 168.91 0) (unit 1)
+  (symbol (lib_id "power:PWR_FLAG") (at 26.035 168.91 0) (unit 1)
     (in_bom yes) (on_board yes) (dnp no)
-    (property "Reference" "#FLG04" (at 40.64 167.005 0)
+    (property "Reference" "#FLG04" (at 26.035 167.005 0)
       (effects (font (size 1.27 1.27)) hide)
     )
-    (property "Value" "PWR_FLAG" (at 36.195 164.465 0)
+    (property "Value" "PWR_FLAG" (at 21.59 164.465 0)
       (effects (font (size 1.27 1.27)) (justify left))
     )
-    (property "Footprint" "" (at 40.64 168.91 0)
+    (property "Footprint" "" (at 26.035 168.91 0)
       (effects (font (size 1.27 1.27)) hide)
     )
-    (property "Datasheet" "~" (at 40.64 168.91 0)
+    (property "Datasheet" "~" (at 26.035 168.91 0)
       (effects (font (size 1.27 1.27)) hide)
     )
@@
     )
   )
-  (sheet (at 95.25 149.225) (size 64.77 40.005)
+  (sheet (at 99.06 150.495) (size 64.77 40.005)
     (stroke (width 0.1524) (type solid))
     (fill (color 0 0 0 0.0000))
-    (property "Sheetname" "Peripherals" (at 95.25 148.59 0)
+    (property "Sheetname" "Peripherals" (at 99.06 149.86 0)
       (effects (font (size 1.27 1.27)) (justify left bottom))
     )
-    (property "Sheetfile" "peripherals.kicad_sch" (at 95.25 189.8146 0)
+    (property "Sheetfile" "peripherals.kicad_sch" (at 99.06 191.0846 0)
       (effects (font (size 1.27 1.27)) (justify left top))
     )
