File: hardware/nextgen/z80ctrlng.kicad_sch (KiCad schematic)
At the start: 33 parts, among them J1 RCBUS, SW1 RESET, SW2 BANK_EN, U1 AS6C4008-55PCN, U2 AVR128DB64x-xPT, U3 74HCT574, U4 74HCT257, U7 AMS1117-3.3

Commit message: Get rid of serial bus links, make banking software controllable
Parts:
- removed JP12: RXB, Jumper:SolderJumper-3_P1.3mm_Open_RoundedPad1.0x1.5mm, symbol Jumper:Jumper_3_Open
- removed JP14: CTS, Jumper:SolderJumper-3_P1.3mm_Bridged12_RoundedPad1.0x1.5mm, symbol Jumper:Jumper_3_Bridged12
- removed JP4: TXB, Jumper:SolderJumper-3_P1.3mm_Open_RoundedPad1.0x1.5mm, symbol Jumper:Jumper_3_Open
- removed JP5: RTS, Jumper:SolderJumper-3_P1.3mm_Bridged12_RoundedPad1.0x1.5mm, symbol Jumper:Jumper_3_Bridged12
- removed SW2: BANK_EN, SamacSys_Parts:JS202011CQN, symbol Switch:SW_DPDT_x2
- removed U3: 74HCT574, Package_DIP:DIP-20_W7.62mm, symbol 74xx:74HCT574
- added C19: 0.1uf, Capacitor_SMD:C_0402_1005Metric, symbol Device:C_Small
- added U3: 74HCT573, Package_SO:TSSOP-20_4.4x6.5mm_P0.65mm, symbol 74xx:74LS573
- added U8: 74LVC1G126, Package_TO_SOT_SMD:SOT-353_SC-70-5, symbol 74xGxx:74LVC1G126
- U4: value 74HCT257 -> 74HC257; footprint Package_DIP:DIP-16_W7.62mm -> Package_SO:SOIC-16_3.9x9.9mm_P1.27mm; now fitted
- renumbered U7 to U5
Connections:
- net BCK is gone; now on net ~{CTS}: U2.47 (PF3)
- net RXB is gone; now on net ~{INT}: U2.13 (PB5)
- net TXB is gone; now on net ~{Z80RST}: U2.12 (PB4)
- net +5V: now also C19.1, U3.20 (VCC), U8.5 (VCC)
- net A15: now also U8.4
- net A15B: now also U8.2
- net A16: now also U2.3 (PA5); no longer U2.44 (XTAL32K1/PF0)
- net A17: now also U2.4 (PA6); no longer U2.45 (XTAL32K2/PF1)
- net A18: now also U2.5 (PA7); no longer U2.46 (PF2)
- net BA15: now also U3.19 (Q0)
- net BA16: now also U3.18 (Q1)
- net BA17: now also U3.17 (Q2)
- net BA18: now also U3.16 (Q3)
- net BB15: now also U3.15 (Q4)
- net BB16: now also U3.14 (Q5)
- net BB17: now also U3.13 (Q6)
- net BB18: now also U3.12 (Q7)
- net D0: now also U3.2 (D0)
- net D1: now also U3.3 (D1)
- net D2: now also U3.4 (D2)
- net D3: now also U3.5 (D3)
- net D4: now also U3.6 (D4)
- net D5: now also U3.7 (D5)
- net D6: now also U3.8 (D6)
- net D7: now also U3.9 (D7)
- net GND: now also C19.2, U3.1 (OE), U3.10 (GND), U8.3 (GND)
- net ~{BANK}: now also U2.44 (XTAL32K1/PF0), U8.1
- net ~{BUSACK}: now also U2.1 (PA3); no longer U2.3 (PA5)
- net ~{HALT}: now also U2.2 (PA4); no longer U2.5 (PA7)
- net ~{INT}: no longer U2.4 (PA6)
- net ~{RD}: now also U2.14 (PB6); no longer U2.2 (PA4)
- net ~{SDCS}: now also U2.46 (PF2); no longer U2.14 (PB6)
- net ~{Z80RST}: no longer U2.1 (PA3)
- new net BLAT: U2.45 (XTAL32K2/PF1), U3.11 (Load)
- no-connect marks 25 -> 28
Other:
- moved on the sheet: C7, C8
